File: keybert/keybert.kicad_pcb (KiCad board)
At the start: 2 copper layers, 146.8 x 123 mm, 62 parts, among them J0 TRRS

Commit message: chore: add yet more to the start of this repo
Before this is ready to be initially presented to the world, all of
the licensing should be fully documented and complied with

fix: typos in the readme

chore: add more license information, fix warranty

This should now be reflective of all of the licensing information I
want included directly within the specification files as well as
CERN OSH recommended header in the one place it can go: the README
Other:
- board text added: "Copyright Travis W Rigg"
- board text added: "Keybert"
- board text added: "Licensed under CERN-OHL-P v2 or later (https://cern.ch/cern-ohl)"
- board text added: "https://github.com/riggtravis/keybert"
Changed lines of the file:
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@@
   )
   (paper "A4")
+  (title_block
+    (title "Keybert")
+    (date "2022-05-16")
+    (rev "0.0.1a")
+    (comment 1 "Copyright Travis W Rigg")
+    (comment 2 "Licensed under CERN-OHL-P v2 or later (https://cern.ch/cern-ohl)")
+    (comment 3 "Repo: https://github.com/riggtravis/keybert")
+  )
   (layers
     (0 "F.Cu" signal)
@@
       (outputformat 1)
       (mirror false)
-      (drillshape 1)
+      (drillshape 0)
       (scaleselection 1)
       (outputdirectory "")
@@
   (gr_line (start 14.44625 18.0975) (end 14.44625 22.86) (layer "Edge.Cuts") (width 0.1))
   (gr_arc (start 156.5275 13.335) (mid 159.895096 14.729904) (end 161.29 18.0975) (layer "Edge.Cuts") (width 0.1))
+  (gr_text "Licensed under CERN-OHL-P v2 or later\n(https://cern.ch/cern-ohl)" (at 129.38125 61.9125) (layer "B.SilkS")
+    (effects (font (size 1 1) (thickness 0.15)) (justify mirror))
+  )
+  (gr_text "https://github.com/riggtravis/keybert" (at 117.475 132.55625) (layer "B.SilkS")
+    (effects (font (size 1 1) (thickness 0.15)) (justify mirror))
+  )
+  (gr_text "Copyright Travis W Rigg" (at 123.03125 54.76875) (layer "B.SilkS")
+    (effects (font (size 1 1) (thickness 0.15)) (justify mirror))
+  )
+  (gr_text "Keybert" (at 150.01875 134.9375) (layer "B.SilkS")
+    (effects (font (size 1 1) (thickness 0.15)) (justify mirror))
+  )
+  (gr_text "Licensed under CERN-OHL-P v2 or later\n(https://cern.ch/cern-ohl)" (at 129.38125 57.94375) (layer "F.SilkS")
+    (effects (font (size 1 1) (thickness 0.15)))
+  )
+  (gr_text "Copyright Travis W Rigg" (at 123.03125 52.3875) (layer "F.SilkS")
+    (effects (font (size 1 1) (thickness 0.15)))
+  )
+  (gr_text "Keybert" (at 155.575 134.9375) (layer "F.SilkS")
+    (effects (font (size 1 1) (thickness 0.15)))
+  )
+  (gr_text "https://github.com/riggtravis/keybert" (at 112.7125 134.9375) (layer "F.SilkS")
+    (effects (font (size 1 1) (thickness 0.15)))
+  )
   (segment (start 114.45875 29.5275) (end 116.99875 29.5275) (width 0.25) (layer "F.Cu") (net 1))
   (segment (start 27.28 22.45) (end 41.1 22.45) (width 0.25) (layer "F.Cu") (net 1))
